File: RTC-zero-SHIM.sch (EAGLE design)
At the start: 16 parts, among them IC1 DS3231/SO, IC2 DS3231M

Commit message: Simplified document names. Generated PDF schematics.
Other:
- note added: "PI-RTCZS-0010"
- note removed: "PI-RTCZEROSHIM-0010"
Changed lines of the file:
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@@
 <plain>
 <text x="256.54" y="7.62" size="2.54" layer="94">1.0</text>
-<text x="198.12" y="7.62" size="2.54" layer="94">PI-RTCZEROSHIM-0010</text>
+<text x="198.12" y="7.62" size="2.54" layer="94">PI-RTCZS-0010</text>
 <text x="165.1" y="25.4" size="2.54" layer="94">Pi Zero sized RTC-SHIM for Pi's 40-pin extension slot
 (c) Andriy Golovnya</text>

Commit message: Added second batter holder as alternative. Generated CAM. Generated PDF schematics. Generated PNG preview image.
Parts:
- added BAT1: CR1220-2, CR1220-2:CR1220-2
Connections:
- net GND: now also BAT1.BAT-
- net VBAT: now also BAT1.BAT+
Changed lines of the file:
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@@
 <part name="GND10" library="SparkFun-PowerSymbols" library_urn="urn:adsk.eagle:library:530" deviceset="GND" device=""/>
 <part name="LOGO4" library="_my_logos" deviceset="MFDECLOGO" device="_L_10MM" value="MFDECLOGO_L_10MM"/>
+<part name="BAT1" library="CR1220-2" deviceset="CR1220-2" device=""/>
+<part name="GND5" library="SparkFun-PowerSymbols" library_urn="urn:adsk.eagle:library:530" deviceset="GND" device=""/>
 </parts>
 <sheets>
@@
 <text x="208.28" y="60.96" size="2.54" layer="94">I2C1 is connected
 by default</text>
-<text x="210.82" y="127" size="2.54" layer="94">Battery holder</text>
+<text x="210.82" y="137.16" size="2.54" layer="94">Battery holder</text>
 <text x="38.1" y="99.06" size="2.54" layer="94">Alternative footprint</text>
 </plain>
@@
 </instance>
 <instance part="LOGO4" gate="G$1" x="106.68" y="2.54" smashed="yes"/>
+<instance part="BAT1" gate="G$1" x="220.98" y="129.54" smashed="yes">
+<attribute name="NAME" x="218.44" y="132.08" size="1.778" layer="96"/>
+<attribute name="VALUE" x="215.9" y="124.46" size="1.778" layer="96"/>
+</instance>
+<instance part="GND5" gate="1" x="231.14" y="127" smashed="yes">
+<attribute name="VALUE" x="231.14" y="126.746" size="1.778" layer="96" align="top-center"/>
+</instance>
 </instances>
 <busses>
@@
 <wire x1="63.5" y1="81.28" x2="71.12" y2="81.28" width="0.1524" layer="91"/>
 <label x="66.04" y="81.28" size="1.778" layer="95"/>
+</segment>
+<segment>
+<pinref part="BAT1" gate="G$1" pin="BAT+"/>
+<wire x1="218.44" y1="129.54" x2="210.82" y2="129.54" width="0.1524" layer="91"/>
+<label x="208.28" y="129.54" size="1.778" layer="95"/>
 </segment>
 </net>
@@
 <pinref part="GND10" gate="1" pin="GND"/>
 </segment>
-</net>
+<segment>
+<pinref part="BAT1" gate="G$1" pin="BAT-"/>
+<wire x1="226.06" y1="129.54" x2="231.14" y2="129.54" width="0.1524" layer="91"/>
+<pinref part="GND5" gate="1" pin="GND"/>
+</segment>
+</net>
