File: RTC-mini-flip-SHIM.sch (EAGLE design)
At the start: 12 parts, among them IC1 DS3231/SO, IC2 DS3231M

Commit message: Moved battery socket to another side to not collide with CPU heat sink. Generated CAM files.
Other:
- note added: "1.1"
- note added: "PI-RTCMS-0011"
- note removed: "1.0"
- note removed: "PI-RTCMS-0010"
Changed lines of the file:
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@@
 <sheet>
 <plain>
-<text x="256.54" y="7.62" size="2.54" layer="94">1.0</text>
-<text x="198.12" y="7.62" size="2.54" layer="94">PI-RTCMS-0010</text>
+<text x="256.54" y="7.62" size="2.54" layer="94">1.1</text>
+<text x="198.12" y="7.62" size="2.54" layer="94">PI-RTCMS-0011</text>
 <text x="165.1" y="25.4" size="2.54" layer="94">Double-mount RTC-mini-flip-SHIM for Pi's extension slot
 (c) Andriy Golovnya</text>
